Commit message: Fix urdf files

File: urdf/turtlebot3_burger.urdf.xacro (robot description, xacro)
@@ -34,10 +34,10 @@
     <parent link="base_link"/>
     <child link="wheel_left_link"/>
-    <origin xyz="0.0 0.08 0.023" rpy="${-M_PI*0.5} 0 0"/>
+    <origin xyz="0.0 0.08 0.023" rpy="${-pi*0.5} 0 0"/>
     <axis xyz="0 0 1"/>
   </joint>
   <link name="wheel_left_link">
     <visual>
-      <origin xyz="0 0 0" rpy="${M_PI*0.5} 0 0"/>
+      <origin xyz="0 0 0" rpy="${pi*0.5} 0 0"/>
       <geometry>
         <mesh filename="package://turtlebot3_description/meshes/wheels/left_tire.stl" scale="0.001 0.001 0.001"/>
@@ -62,10 +62,10 @@
     <parent link="base_link"/>
     <child link="wheel_right_link"/>
-    <origin xyz="0.0 -0.08 0.023" rpy="${-M_PI*0.5} 0 0"/>
+    <origin xyz="0.0 -0.08 0.023" rpy="${-pi*0.5} 0 0"/>
     <axis xyz="0 0 1"/>
   </joint>
   <link name="wheel_right_link">
     <visual>
-      <origin xyz="0 0 0" rpy="${M_PI*0.5} 0 0"/>
+      <origin xyz="0 0 0" rpy="${pi*0.5} 0 0"/>
       <geometry>
         <mesh filename="package://turtlebot3_description/meshes/wheels/right_tire.stl" scale="0.001 0.001 0.001"/>
@@ -90,5 +90,5 @@
     <parent link="base_link"/>
     <child link="caster_back_link"/>
-    <origin xyz="-0.081 0 -0.004" rpy="${-M_PI*0.5} 0 0"/>
+    <origin xyz="-0.081 0 -0.004" rpy="${-pi*0.5} 0 0"/>
   </joint>
   <link name="caster_back_link">

File: urdf/turtlebot3_burger_noisy_scan.urdf.xacro (robot description, xacro)
@@ -34,10 +34,10 @@
     <parent link="base_link"/>
     <child link="wheel_left_link"/>
-    <origin xyz="0.0 0.08 0.023" rpy="${-M_PI*0.5} 0 0"/>
+    <origin xyz="0.0 0.08 0.023" rpy="${-pi*0.5} 0 0"/>
     <axis xyz="0 0 1"/>
   </joint>
   <link name="wheel_left_link">
     <visual>
-      <origin xyz="0 0 0" rpy="${M_PI*0.5} 0 0"/>
+      <origin xyz="0 0 0" rpy="${pi*0.5} 0 0"/>
       <geometry>
         <mesh filename="package://turtlebot3_description/meshes/wheels/left_tire.stl" scale="0.001 0.001 0.001"/>
@@ -62,10 +62,10 @@
     <parent link="base_link"/>
     <child link="wheel_right_link"/>
-    <origin xyz="0.0 -0.08 0.023" rpy="${-M_PI*0.5} 0 0"/>
+    <origin xyz="0.0 -0.08 0.023" rpy="${-pi*0.5} 0 0"/>
     <axis xyz="0 0 1"/>
   </joint>
   <link name="wheel_right_link">
     <visual>
-      <origin xyz="0 0 0" rpy="${M_PI*0.5} 0 0"/>
+      <origin xyz="0 0 0" rpy="${pi*0.5} 0 0"/>
       <geometry>
         <mesh filename="package://turtlebot3_description/meshes/wheels/right_tire.stl" scale="0.001 0.001 0.001"/>
@@ -90,5 +90,5 @@
     <parent link="base_link"/>
     <child link="caster_back_link"/>
-    <origin xyz="-0.081 0 -0.004" rpy="${-M_PI*0.5} 0 0"/>
+    <origin xyz="-0.081 0 -0.004" rpy="${-pi*0.5} 0 0"/>
   </joint>
   <link name="caster_back_link">

File: urdf/turtlebot3_burger_restricted_scan.urdf.xacro (robot description, xacro)
@@ -34,10 +34,10 @@
     <parent link="base_link"/>
     <child link="wheel_left_link"/>
-    <origin xyz="0.0 0.08 0.023" rpy="${-M_PI*0.5} 0 0"/>
+    <origin xyz="0.0 0.08 0.023" rpy="${-pi*0.5} 0 0"/>
     <axis xyz="0 0 1"/>
   </joint>
   <link name="wheel_left_link">
     <visual>
-      <origin xyz="0 0 0" rpy="${M_PI*0.5} 0 0"/>
+      <origin xyz="0 0 0" rpy="${pi*0.5} 0 0"/>
       <geometry>
         <mesh filename="package://turtlebot3_description/meshes/wheels/left_tire.stl" scale="0.001 0.001 0.001"/>
@@ -62,10 +62,10 @@
     <parent link="base_link"/>
     <child link="wheel_right_link"/>
-    <origin xyz="0.0 -0.08 0.023" rpy="${-M_PI*0.5} 0 0"/>
+    <origin xyz="0.0 -0.08 0.023" rpy="${-pi*0.5} 0 0"/>
     <axis xyz="0 0 1"/>
   </joint>
   <link name="wheel_right_link">
     <visual>
-      <origin xyz="0 0 0" rpy="${M_PI*0.5} 0 0"/>
+      <origin xyz="0 0 0" rpy="${pi*0.5} 0 0"/>
       <geometry>
         <mesh filename="package://turtlebot3_description/meshes/wheels/right_tire.stl" scale="0.001 0.001 0.001"/>
@@ -90,5 +90,5 @@
     <parent link="base_link"/>
     <child link="caster_back_link"/>
-    <origin xyz="-0.081 0 -0.004" rpy="${-M_PI*0.5} 0 0"/>
+    <origin xyz="-0.081 0 -0.004" rpy="${-pi*0.5} 0 0"/>
   </joint>
   <link name="caster_back_link">
