Commit message: Major revision changes to simplify the repo structure. Major rewrites to launch files.

File: urdf/asl_turtlebot.gazebo.xacro (robot description, xacro)
@@ -8,4 +8,5 @@
       <odometryTopic>odom</odometryTopic>
       <odometryFrame>odom</odometryFrame>
+      <publishTf>true</publishTf>
       <robotBaseFrame>base_footprint</robotBaseFrame>
       <publishWheelTF>false</publishWheelTF>

File: urdf/asl_turtlebot.urdf.xacro (robot description, xacro)
@@ -2,5 +2,5 @@
 <robot name="turtlebot3_burger" xmlns:xacro="http://ros.org/wiki/xacro">
   <xacro:include filename="$(find turtlebot3_description)/urdf/common_properties.xacro"/>
-  <xacro:include filename="$(find asl_turtlebot)/urdf/turtlebot3_burger.gazebo.xacro"/>
+  <xacro:include filename="$(find asl_turtlebot)/urdf/asl_turtlebot.gazebo.xacro"/>
   <link name="base_footprint"/>
   <joint name="base_joint" type="fixed">
@@ -146,4 +146,5 @@
         <box size=".1 .1 .1"/>
       </geometry>
+      <material name="red"/>
     </visual>
     <collision>
@@ -164,78 +165,3 @@
     <origin xyz="-0.032 0 0.198" rpy="0 0 0"/>
   </joint>
-  <link name="right_gripper">
-    <visual>
-      <origin xyz="0.05 0 0" rpy="0 0 0"/>
-      <geometry>
-        <box size=".1 .02 .02"/>
-      </geometry>
-      <material name="red"/>
-    </visual>
-    <collision>
-      <origin xyz="0.05 0 0" rpy="0 0 0"/>
-      <geometry>
-        <box size=".1 .02 .02"/>
-      </geometry>
-    </collision>
-    <inertial>
-      <mass value="1e-2"/>
-      <origin xyz="0 0 0" rpy="0 0 0"/>
-      <inertia ixx="1e-2" iyy="1e-3" izz="1e-2" ixy="0" ixz="0" iyz="0"/>
-    </inertial>
-  </link>
-  <link name="left_gripper">
-    <visual>
-      <origin xyz="0.05 0 0" rpy="0 0 0"/>
-      <geometry>
-        <box size=".1 .02 .02"/>
-      </geometry>
-      <material name="red"/>
-    </visual>
-    <collision>
-      <origin xyz="0.05 0 0" rpy="0 0 0"/>
-      <geometry>
-        <box size=".1 .02 .02"/>
-      </geometry>
-    </collision>
-    <inertial>
-      <mass value="1e-2"/>
-      <origin xyz="0 0 0" rpy="0 0 0"/>
-      <inertia ixx="1e-2" iyy="1e-3" izz="1e-2" ixy="0" ixz="0" iyz="0"/>
-    </inertial>
-  </link>
-  <joint name="right_gripper_joint" type="prismatic">
-    <parent link="base_link"/>
-    <child link="right_gripper"/>
-    <axis xyz="0 -1 0"/>
-    <origin xyz="0.05 -0.01 0.03" rpy="0 0 0"/>
-    <limit lower="0" upper=".03" velocity=".1" effort="100"/>
-  </joint>
-  <joint name="left_gripper_joint" type="prismatic">
-    <parent link="base_link"/>
-    <child link="left_gripper"/>
-    <axis xyz="0 1 0"/>
-    <origin xyz="0.05 0.01 0.03" rpy="0 0 0"/>
-    <mimic joint="right_gripper_joint" multiplier="1"/>
-    <limit lower="0" upper=".03" velocity=".1" effort="100"/>
-  </joint>
-  <transmission name="right_gripper_trans">
-    <type>transmission_interface/SimpleTransmission</type>
-    <joint name="right_gripper_joint">
-      <hardwareInterface>hardware_interface/EffortJointInterface</hardwareInterface>
-    </joint>
-    <actuator name="right_gripper_motor">
-      <hardwareInterface>hardware_interface/EffortJointInterface</hardwareInterface>
-      <mechanicalReduction>1</mechanicalReduction>
-    </actuator>
-  </transmission>
-  <transmission name="left_gripper_trans">
-    <type>transmission_interface/SimpleTransmission</type>
-    <joint name="left_gripper_joint">
-      <hardwareInterface>hardware_interface/EffortJointInterface</hardwareInterface>
-    </joint>
-    <actuator name="left_gripper_motor">
-      <hardwareInterface>hardware_interface/EffortJointInterface</hardwareInterface>
-      <mechanicalReduction>1</mechanicalReduction>
-    </actuator>
-  </transmission>
 </robot>

File: urdf/asl_turtlebot_gripper.urdf.xacro (robot description, xacro)
@@ -2,5 +2,5 @@
 <robot name="turtlebot3_burger" xmlns:xacro="http://ros.org/wiki/xacro">
   <xacro:include filename="$(find turtlebot3_description)/urdf/common_properties.xacro"/>
-  <xacro:include filename="$(find asl_turtlebot)/urdf/turtlebot3_burger_restricted_scan.gazebo.xacro"/>
+  <xacro:include filename="$(find asl_turtlebot)/urdf/asl_turtlebot.gazebo.xacro"/>
   <link name="base_footprint"/>
   <joint name="base_joint" type="fixed">
@@ -146,5 +146,4 @@
         <box size=".1 .1 .1"/>
       </geometry>
-      <material name="red"/>
     </visual>
     <collision>
@@ -165,3 +164,78 @@
     <origin xyz="-0.032 0 0.198" rpy="0 0 0"/>
   </joint>
+  <link name="right_gripper">
+    <visual>
+      <origin xyz="0.05 0 0" rpy="0 0 0"/>
+      <geometry>
+        <box size=".1 .02 .02"/>
+      </geometry>
+      <material name="red"/>
+    </visual>
+    <collision>
+      <origin xyz="0.05 0 0" rpy="0 0 0"/>
+      <geometry>
+        <box size=".1 .02 .02"/>
+      </geometry>
+    </collision>
+    <inertial>
+      <mass value="1e-2"/>
+      <origin xyz="0 0 0" rpy="0 0 0"/>
+      <inertia ixx="1e-2" iyy="1e-3" izz="1e-2" ixy="0" ixz="0" iyz="0"/>
+    </inertial>
+  </link>
+  <link name="left_gripper">
+    <visual>
+      <origin xyz="0.05 0 0" rpy="0 0 0"/>
+      <geometry>
+        <box size=".1 .02 .02"/>
+      </geometry>
+      <material name="red"/>
+    </visual>
+    <collision>
+      <origin xyz="0.05 0 0" rpy="0 0 0"/>
+      <geometry>
+        <box size=".1 .02 .02"/>
+      </geometry>
+    </collision>
+    <inertial>
+      <mass value="1e-2"/>
+      <origin xyz="0 0 0" rpy="0 0 0"/>
+      <inertia ixx="1e-2" iyy="1e-3" izz="1e-2" ixy="0" ixz="0" iyz="0"/>
+    </inertial>
+  </link>
+  <joint name="right_gripper_joint" type="prismatic">
+    <parent link="base_link"/>
+    <child link="right_gripper"/>
+    <axis xyz="0 -1 0"/>
+    <origin xyz="0.05 -0.01 0.03" rpy="0 0 0"/>
+    <limit lower="0" upper=".03" velocity=".1" effort="100"/>
+  </joint>
+  <joint name="left_gripper_joint" type="prismatic">
+    <parent link="base_link"/>
+    <child link="left_gripper"/>
+    <axis xyz="0 1 0"/>
+    <origin xyz="0.05 0.01 0.03" rpy="0 0 0"/>
+    <mimic joint="right_gripper_joint" multiplier="1"/>
+    <limit lower="0" upper=".03" velocity=".1" effort="100"/>
+  </joint>
+  <transmission name="right_gripper_trans">
+    <type>transmission_interface/SimpleTransmission</type>
+    <joint name="right_gripper_joint">
+      <hardwareInterface>hardware_interface/EffortJointInterface</hardwareInterface>
+    </joint>
+    <actuator name="right_gripper_motor">
+      <hardwareInterface>hardware_interface/EffortJointInterface</hardwareInterface>
+      <mechanicalReduction>1</mechanicalReduction>
+    </actuator>
+  </transmission>
+  <transmission name="left_gripper_trans">
+    <type>transmission_interface/SimpleTransmission</type>
+    <joint name="left_gripper_joint">
+      <hardwareInterface>hardware_interface/EffortJointInterface</hardwareInterface>
+    </joint>
+    <actuator name="left_gripper_motor">
+      <hardwareInterface>hardware_interface/EffortJointInterface</hardwareInterface>
+      <mechanicalReduction>1</mechanicalReduction>
+    </actuator>
+  </transmission>
 </robot>

File: urdf/asl_turtlebot_hw4_arena.urdf.xacro (robot description, xacro)
@@ -2,5 +2,5 @@
 <robot name="turtlebot3_burger" xmlns:xacro="http://ros.org/wiki/xacro">
   <xacro:include filename="$(find turtlebot3_description)/urdf/common_properties.xacro"/>
-  <xacro:include filename="$(find asl_turtlebot)/urdf/turtlebot3_burger.gazebo.xacro"/>
+  <xacro:include filename="$(find asl_turtlebot)/urdf/asl_turtlebot_hw4_arena.gazebo.xacro"/>
   <link name="base_footprint"/>
   <joint name="base_joint" type="fixed">

File: urdf/asl_turtlebot_hw4_maze.urdf.xacro (robot description, xacro)
@@ -2,5 +2,5 @@
 <robot name="turtlebot3_burger" xmlns:xacro="http://ros.org/wiki/xacro">
   <xacro:include filename="$(find turtlebot3_description)/urdf/common_properties.xacro"/>
-  <xacro:include filename="$(find asl_turtlebot)/urdf/turtlebot3_burger_noisy_scan.gazebo.xacro"/>
+  <xacro:include filename="$(find asl_turtlebot)/urdf/asl_turtlebot_hw4_maze.gazebo.xacro"/>
   <link name="base_footprint"/>
   <joint name="base_joint" type="fixed">
